File: Hard/Barometer.sch (KiCad schematic (older format))
At the start: 55 parts, among them J2 KRC_Conn_SWD, J3 USB_B_Micro, J4 KRC_Conn_CAN, U1 CY8C58xxLTI-LPxxx, U2 W25N01GVxxIG-IT, U3 NCV7342, U4 LPS22HB, Y1 24MHz

Commit message: [update] 回路図のフィールドを編集
Parts:
- C28, D4, D5: Agency 秋月電子 -> akizuki
- U4: Agency (none) -> Digikey; Link (none) -> https://www.digikey.jp/product-detail/ja/stmicroelectronics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; MPN (none) -> LPS22HB
Changed lines of the file:
@@
 F 2 "Package_LGA:ST_HLGA-10_2.5x2.5mm_P0.6mm_LayoutBorder3x2y" H 5000 6750 50  0001 C CNN
 F 3 "www.st.com/resource/en/datasheet/lps25hb.pdf" H 5050 6600 50  0001 C CNN
+F 4 "Digikey" H 0   0   50  0001 C CNN "Agency"
+F 5 "https://www.digikey.jp/product-detail/ja/stmicroelectronics/LPS22HBTR/497-16265-1-ND/5799917" H 0   0   50  0001 C CNN "Link"
+F 6 "LPS22HB" H 0   0   50  0001 C CNN "MPN"
 	1    5000 6950
 	1    0    0    -1
@@
 F 2 "Capacitor_SMD:C_0603_1608Metric" H 4450 6350 50  0001 C CNN
 F 3 "https://search.murata.co.jp/Ceramy/image/img/A01X/G101/ENG/GRM188R6YA106MA73-01.pdf" H 4450 6350 50  0001 C CNN
-F 4 "秋月電子" H 4450 6350 50  0001 C CNN "Agency"
+F 4 "akizuki" H 4450 6350 50  0001 C CNN "Agency"
 F 5 "GRM188R6YA106MA73D" H 4450 6350 50  0001 C CNN "MPN"
 F 6 "10uF" H 4450 6350 50  0001 C CNN "Value"
@@
 F 2 "Diode_SMD:D_TUMD2" V 2250 750 50  0001 C CNN
 F 3 "http://akizukidenshi.com/download/ds/rohm/rsx101vam30-j.pdf" V 2250 750 50  0001 C CNN
-F 4 "秋月電子" H 2250 750 50  0001 C CNN "Agency"
+F 4 "akizuki" H 2250 750 50  0001 C CNN "Agency"
 F 5 "http://akizukidenshi.com/catalog/g/gI-05951/" H 2250 750 50  0001 C CNN "Link"
 F 6 "RSX101VAM-30TR" H 2250 750 50  0001 C CNN "MPN"
@@
 F 2 "Diode_SMD:D_TUMD2" V 2250 1800 50  0001 C CNN
 F 3 "http://akizukidenshi.com/download/ds/rohm/rsx101vam30-j.pdf" V 2250 1800 50  0001 C CNN
-F 4 "秋月電子" H 2250 1800 50  0001 C CNN "Agency"
+F 4 "akizuki" H 2250 1800 50  0001 C CNN "Agency"
 F 5 "http://akizukidenshi.com/catalog/g/gI-05951/" H 2250 1800 50  0001 C CNN "Link"
 F 6 "RSX101VAM-30TR" H 2250 1800 50  0001 C CNN "MPN"
